File: schematic/sw1-2.kicad_sch (KiCad schematic)
At the start: 34 parts, among them Q5 Q_PNP_BRT 20k/20k, Q6 Q_NPN, Q6 Q_NPN_BRT 10k/10k, Q9 Q_NPN, SW1 SW_Push, SW2 SW_Push

Commit message: Minor corrections to sw1-2, renamed duplicate Q6 to Q10
Parts:
- renumbered Q6 to Q10
Connections:
- net GND: now also Q6.E, R44.1
- net LED_CTRL1: now also R49.2; no longer Q9.C
Changed lines of the file:
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@@
 	(text "via to inner layer"
 		(exclude_from_sim no)
-		(at 56.388 75.946 0)
+		(at 53.086 76.708 0)
 		(effects
 			(font
@@
 	(wire
 		(pts
-			(xy 59.69 71.12) (xy 72.39 71.12)
+			(xy 59.69 71.12) (xy 67.31 71.12)
 		)
 		(stroke
@@
 		)
 	)
-	(global_label "LED_CTRL1"
-		(shape output)
-		(at 55.88 78.74 0)
+	(global_label "PP2"
+		(shape input)
+		(at 26.67 34.29 180)
 		(fields_autoplaced yes)
 		(effects
@@
 				(size 1.27 1.27)
 			)
-			(justify left)
+			(justify right)
 		)
 		(property "Intersheetrefs" "${INTERSHEET_REFS}"
-			(at 69.0251 78.74 0)
+			(at 19.9353 34.29 0)
 			(effects
 				(font
 					(size 1.27 1.27)
 				)
-				(justify left)
+				(justify right)
 				(hide yes)
 			)
 		)
 	)
-	(global_label "PP2"
+	(global_label "KWL0{slash}PL0"
 		(shape input)
-		(at 26.67 34.29 180)
+		(at 130.81 22.86 0)
 		(fields_autoplaced yes)
 		(effects
@@
 				(size 1.27 1.27)
 			)
-			(justify right)
+			(justify left)
 		)
 		(property "Intersheetrefs" "${INTERSHEET_REFS}"
-			(at 19.9353 34.29 0)
+			(at 143.5923 22.86 0)
 			(effects
 				(font
 					(size 1.27 1.27)
 				)
-				(justify right)
+				(justify left)
 				(hide yes)
 			)
 		)
 	)
-	(global_label "KWL0{slash}PL0"
+	(global_label "LED_CTRL1"
 		(shape input)
-		(at 130.81 22.86 0)
+		(at 67.31 71.12 0)
 		(fields_autoplaced yes)
 		(effects
@@
 		)
 		(property "Intersheetrefs" "${INTERSHEET_REFS}"
-			(at 143.5923 22.86 0)
+			(at 80.4551 71.12 0)
 			(effects
 				(font
@@
 	)
 	(symbol
+		(lib_id "power:GND")
+		(at 26.67 45.72 0)
+		(unit 1)
+		(exclude_from_sim no)
+		(in_bom yes)
+		(on_board yes)
+		(dnp no)
+		(fields_autoplaced yes)
+		(property "Reference" "#PWR026"
+			(at 26.67 52.07 0)
+			(effects
+				(font
+					(size 1.27 1.27)
+				)
+				(hide yes)
+			)
+		)
+		(property "Value" "GND"
+			(at 26.67 50.8 0)
+			(effects
+				(font
+					(size 1.27 1.27)
+				)
+			)
+		)
+		(property "Footprint" ""
+			(at 26.67 45.72 0)
+			(effects
+				(font
+					(size 1.27 1.27)
+				)
+				(hide yes)
+			)
+		)
+		(property "Datasheet" ""
+			(at 26.67 45.72 0)
+			(effects
+				(font
+					(size 1.27 1.27)
+				)
+				(hide yes)
+			)
+		)
+		(property "Description" "Power symbol creates a global label with name \"GND\" , ground"
+			(at 26.67 45.72 0)
+			(effects
+				(font
+					(size 1.27 1.27)
+				)
+				(hide yes)
+			)
+		)
+		(pin "1"
+		)
+		(instances
+			(project ""
+				(path "/9b2d5e25-09e0-4218-be17-c115a885c472/a96c1825-69cc-4d78-b19f-6fdfeb00d9a9"
+					(reference "#PWR026")
+					(unit 1)
+				)
+			)
+		)
+	)
+	(symbol
 		(lib_id "Device:Q_NPN_BRT")
 		(at 46.99 34.29 0)
@@
 		(dnp yes)
 		(fields_autoplaced yes)
-		(property "Reference" "Q6"
+		(property "Reference" "Q10"
 			(at 116.84 71.1199 0)
 			(effects
@@
 			(project "Preh-13250-0500-L"
 				(path "/9b2d5e25-09e0-4218-be17-c115a885c472/a96c1825-69cc-4d78-b19f-6fdfeb00d9a9"
-					(reference "Q6")
+					(reference "Q10")
 					(unit 1)
 				)

Commit message: Added J5 and assoc. resistor network. Added traceable signals for MYSTERY_SIG
Parts:
- Q10: now fitted
- R36: value R -> 85k
Connections:
- net +VBATT_PROT: now also Q5.E; no longer Q5.C
- net at R23.2, R24.2: now also Q5.C; no longer Q5.B
- net at Q6.C: now also Q5.B; no longer Q5.E
Other:
- note added: "Partially populated for 3G0 update"
- note added: "may be through 1 or 2 resistors, see general sheet"
- note removed: "Unpopulated on top-right of sec side"
- moved on the sheet: C10, Q5, Q6
